File: PDB-KiCad10/PowerDistributionBoard.kicad_sch (KiCad schematic)
At the start: 14 parts, among them U1 XL4016, U3 AMS1117

Commit message: Upgraded the schematic
Parts:
- removed R4: 1k, symbol Device:R
- removed U3: AMS1117, Package_TO_SOT_SMD:SOT-223-3_TabPin2, symbol Regulator_Linear:AMS1117
- added C7: 1uF, symbol Device:C
- added J2: Main Input, symbol Connector:Screw_Terminal_01x02
- added J3: Main Output, symbol Connector:Screw_Terminal_01x02
- added J4: USB_A, Connector_USB:USB_A_Molex_67643_Horizontal, symbol Connector:USB_A
- added J5, J6: USB_C_Receptacle_PowerOnly_6P, symbol Connector:USB_C_Receptacle_PowerOnly_6P
- added J7: Conn_01x04, symbol Connector_Generic:Conn_01x04
- added SW1, SW2: SW_Push, symbol Switch:SW_Push
- added U2: AMS1117-3.3, Package_TO_SOT_SMD:SOT-223-3_TabPin2, symbol Regulator_Linear:AMS1117-3.3
- added U3: ESP32-WROOM-32E, RF_Module:ESP32-WROOM-32D, symbol RF_Module:ESP32-WROOM-32E
- added U4: FUSB302BMPX, Package_DFN_QFN:WQFN-14-1EP_2.5x2.5mm_P0.5mm_EP1.45x1.45mm, symbol Interface_USB:FUSB302BMPX
- C1: value C_Polarized -> 470uF 50V
- C2: value C_Polarized -> 470uF 16V
- C3: value C -> 0.1uF/100nF
- C4: value C -> 0.1uF / 100nF
- D1: value D_Schottky -> D_Schottky(MBR1545)
- L1: value L -> 47uH (8A+)
- R3: value 2k -> 10K
Connections:
- net +24V: now also J2.2 (Pin_2), J3.1 (Pin_1)
- net +3.3V: now also R3.1, J7.1 (Pin_1), U2.2 (VO), U3.2 (VDD); no longer R3.2
- net +5V: now also J4.1 (VBUS), J5.A9 (VBUS), J5.B9 (VBUS), J6.A9 (VBUS), J6.B9 (VBUS), U2.3 (VI)
- net GND: now also C7.2, J2.1 (Pin_1), J3.2 (Pin_2), J4.4 (GND), J4.SH (Shield), J5.A12 (GND), J5.B12 (GND), J5.SH (SHIELD), J6.A12 (GND), J6.B12 (GND), J6.SH (SHIELD), J7.4 (Pin_4), SW1.2, SW2.2, U2.1 (GND), U3.1 (GND), U3.15 (GND), U3.38 (GND), U3.39 (GND)
- new net: C7.1, R3.2, SW1.1, U3.3 (EN)
- new net: U4.1 (CC2), U4.14 (CC2)
- new net: U4.10 (CC1), U4.11 (CC1)
- new net: U4.15 (GND), U4.8 (GND), U4.9 (GND)
- new net: U4.3 (VDD), U4.4 (VDD)
- new net: SW2.1, U3.25 (IO0)
- new net RXD0: J7.3 (Pin_3), U3.34 (RXD0/IO3)
- new net TXD0: J7.2 (Pin_2), U3.35 (TXD0/IO1)
- no-connect marks 0 -> 2
Other:
- note added: "MCU"
- note added: "Power Management"
- moved on the sheet: C1, C2, C3, C4, C5, C6, D1, L1, R1, R2, U1

Commit message: Updated Schematic
Parts:
- added C10: 470uF 16V, symbol Device:C_Polarized
- added C8: 0.1uF, symbol Device:C
- added C9: 470uF 50V, symbol Device:C_Polarized
- added D2: D_Schottky, symbol Device:D_Schottky
- added F1: 10A, symbol Device:Fuse
- added L2: 47uH, symbol Device:L
- added Q1: 2N7002(9V), Package_TO_SOT_SMD:SOT-23, symbol Transistor_FET:2N7002
- added Q2: 2N7002(12V), Package_TO_SOT_SMD:SOT-23, symbol Transistor_FET:2N7002
- added R10, R11: R_Shunt, symbol Device:R_Shunt
- added R4, R5: R, symbol Device:R
- added R6: 10k, symbol Device:R
- added R7: 3.3k, symbol Device:R
- added R8: 3k, symbol Device:R
- added R9: 1.74k, symbol Device:R
- added SW3: SW_SPST, symbol Switch:SW_SPST
- added U5: LM2596S-ADJ, Package_TO_SOT_SMD:TO-263-5_TabPin3, symbol Regulator_Switching:LM2596S-ADJ
- added U6, U8: INA226, Package_SO:TSSOP-10_3x3mm_P0.5mm, symbol Sensor_Energy:INA226
- added U7: OLED, OLED:miniOLED, symbol Display_Graphic:ER_OLEDM0.91_1x-I2C
- J5: value USB_C_Receptacle_PowerOnly_6P -> USB_C_Fast_Charging
Connections:
- net +24V: now also C9.1, R10.1, U5.1 (VIN); no longer C1.1, C3.1, J3.1 (Pin_1), U1.1 (VIN)
- net +3.3V: now also U4.3 (VDD), U4.4 (VDD), C8.1, R4.1, R5.1, U6.6 (VS), U7.2 (VCC), U8.2 (A0), U8.6 (VS)
- net +5V: now also U4.12 (VCONN), U4.13 (VCONN); no longer J5.A9 (VBUS), J5.B9 (VBUS)
- net GND: now also U4.15 (GND), U4.8 (GND), U4.9 (GND), C10.2, C8.2, C9.2, D2.2 (A), Q1.2 (S), Q2.2 (S), R7.1, U5.3 (GND), U5.5 (~{ON}/OFF), U6.1 (A1), U6.2 (A0), U6.7 (GND), U7.1 (GND), U8.1 (A1), U8.7 (GND)
- net RXD0: now also U3.35 (TXD0/IO1); no longer U3.34 (RXD0/IO3)
- net TXD0: now also U3.34 (RXD0/IO3); no longer U3.35 (TXD0/IO1)
- net at U4.1 (CC2), U4.14 (CC2): now also J5.A5 (CC1)
- net at U4.10 (CC1), U4.11 (CC1): now also J5.B5 (CC2)
- net VBUS: now reaches U4.2 (VBUS)
- net VBUS: now also J5.A9 (VBUS), J5.B9 (VBUS), R11.1
- net Interupt: now reaches U4.5 (INT_N)
- net Interupt: now also U3.26 (IO4)
- net SCL: now reaches U4.6 (SCL)
- net SCL: now also U3.36 (IO22), R5.2, U6.5 (SCL), U7.3 (SCL), U8.5 (SCL)
- net SDA: now reaches U4.7 (SDA)
- net SDA: now also U3.33 (IO21), R4.2, U6.4 (SDA), U7.4 (SDA), U8.4 (SDA)
- net I012: now reaches U3.14 (IO12)
- net I012: now also Q1.1 (G)
- net I013: now reaches U3.16 (IO13)
- net I013: now also Q2.1 (G)
- new net: C10.1, L2.2, R11.4, R6.2
- new net: D2.1 (K), L2.1, U5.2 (OUT)
- new net: R6.1, R7.2, R8.1, R9.1, U5.4 (FB)
- new net: F1.1, SW3.1 (A)
- new net: J3.1 (Pin_1), SW3.2 (B)
- new net: C1.1, C3.1, F1.2, R10.4, U1.1 (VIN)
- new net: Q1.3 (D), R8.2
- new net: Q2.3 (D), R9.2
- new net VBUS+: R11.3, U8.10 (Vin+), U8.8 (Vbus)
- new net VBUS-: R11.2, U8.9 (Vin-)
- new net VIN+: R10.2, U6.10 (Vin+), U6.8 (Vbus)
- new net VIN-: R10.3, U6.9 (Vin-)
- no-connect marks 2 -> 24
Other:
- note added: "10A limit"
- note added: "Power Analysis"
- note added: "USB Power Only"
- title: (none) -> Power Distribution Board
- moved on the sheet: C1, C2, C3, C4, C5, C6, C7, D1, J2, J3, J4, J6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

Commit message: V1.0 of Schematic is complete
Parts:
- removed J7: Conn_01x04, symbol Connector_Generic:Conn_01x04
- removed U3: ESP32-WROOM-32E, RF_Module:ESP32-WROOM-32D, symbol RF_Module:ESP32-WROOM-32E
- added D3, D4: LED, LED_THT:LED_D3.0mm, symbol Device:LED
- added H1, H2, H3, H4: MountingHole, MountingHole:MountingHole_3.2mm_M3, symbol Mechanical:MountingHole
- added J1: USB_C_Programming_Port, Connector_USB:USB_C_Receptacle_HRO_TYPE-C-31-M-12, symbol Connector:USB_C_Receptacle_USB2.0_16P
- added Q3: AO3401A, Package_TO_SOT_SMD:SOT-23, symbol Transistor_FET:AO3401A
- added Q4: 2N7002, Package_TO_SOT_SMD:SOT-23, symbol Transistor_FET:2N7002
- added R12, R18: 1K, Resistor_SMD:R_0805_2012Metric_Pad1.20x1.40mm_HandSolder, symbol Device:R
- added R13, R14, R17, R19, R20: 10K, Resistor_SMD:R_0805_2012Metric_Pad1.20x1.40mm_HandSolder, symbol Device:R
- added R15, R16: 5.1K, Resistor_SMD:R_0805_2012Metric_Pad1.20x1.40mm_HandSolder, symbol Device:R
- added U3: ESP32-S3-WROOM-1, RF_Module:ESP32-S3-WROOM-1, symbol RF_Module:ESP32-S3-WROOM-1
- C1, C9: footprint (none) -> Capacitor_THT:CP_Radial_D10.0mm_P5.00mm
- C10, C2: footprint (none) -> Capacitor_THT:CP_Radial_D8.0mm_P3.50mm
- C3, C4, C7, C8: footprint (none) -> Capacitor_SMD:C_0805_2012Metric_Pad1.18x1.45mm_HandSolder
- C5, C6: footprint (none) -> Capacitor_THT:CP_Radial_D5.0mm_P2.00mm
- D1: footprint (none) -> Package_TO_SOT_THT:TO-220-2_Vertical
- D2: footprint (none) -> Diode_SMD:D_SMC_Handsoldering
- F1: footprint (none) -> Fuse:Fuseholder_Cylinder-5x20mm_Schurter_0031_8201_Horizontal_Open
- J2, J3: footprint (none) -> TerminalBlock_Phoenix:TerminalBlock_Phoenix_MKDS-1,5-2-5.08_1x02_P5.08mm_Horizontal
- J5: footprint (none) -> Connector_USB:USB_C_Receptacle_HRO_TYPE-C-31-M-12
- J6: footprint (none) -> Connector_USB:USB_C_Receptacle_GCT_USB4125-xx-x_6P_TopMnt_Horizontal
- L1: footprint (none) -> Inductor_THT:L_Toroid_Vertical_L24.6mm_W15.5mm_P11.44mm_Pulse_KM-4
- L2: footprint (none) -> Inductor_SMD:L_12x12mm_H8mm
- R1, R2, R3, R6, R7, R8, R9: footprint (none) -> Resistor_SMD:R_0805_2012Metric_Pad1.20x1.40mm_HandSolder
- R10, R11: footprint (none) -> Resistor_SMD:R_2512_6332Metric_Pad1.40x3.35mm_HandSolder
- R4, R5: value R -> 4.7K; footprint (none) -> Resistor_SMD:R_0805_2012Metric_Pad1.20x1.40mm_HandSolder
- SW1, SW2: footprint (none) -> PDB-KiCad10:SW_PUSH_6x6mm_2Pin_P5.08mm
- SW3: footprint (none) -> Button_Switch_THT:SW_Slide_SPDT_Straight_CK_OS102011MS2Q
Connections:
- net +3.3V: now also U3.2 (3V3)
- net +5V: now also R18.1, R19.2, R20.2
- net GND: now also D3.2 (A), D4.2 (A), J1.A1 (GND), J1.A12 (GND), J1.B1 (GND), J1.B12 (GND), J1.SH (SHIELD), Q4.2 (S), R13.1, R15.2, R16.2, U3.1 (GND), U3.40 (GND), U3.41 (GND)
- net Interupt: now also U3.7 (IO7)
- net SCL: now also U3.17 (IO9)
- net SDA: now also U3.12 (IO8)
- net VBUS: now also Q3.2 (S), R14.2; no longer J5.A9 (VBUS), J5.B9 (VBUS)
- net at C7.1, R3.2, SW1.1: now also U3.3 (EN)
- net at F1.1, SW3.1 (A): now also C1.1, C3.1, U1.1 (VIN)
- net at J3.1 (Pin_1), SW3.2 (B): now also R17.1
- net at SW2.1: now also U3.27 (IO0)
- net at J6.A5 (CC1): now also R19.1
- net at J6.B5 (CC2): now also R20.1
- net I012 renamed I04
- net I04: now also U3.4 (IO4)
- net I013 renamed I05
- net I05: now also U3.5 (IO5)
- new net: F1.2, R10.4
- new net: D3.1 (K), R17.2
- new net: J5.A9 (VBUS), J5.B9 (VBUS), Q3.3 (D)
- new net: Q4.1 (G), R12.1, R13.2
- new net: J1.B5 (CC2), R16.1
- new net: J1.A4 (VBUS), J1.A9 (VBUS), J1.B4 (VBUS), J1.B9 (VBUS)
- new net: J1.A5 (CC1), R15.1
- new net: D4.1 (K), R18.2
- new net IO19: J1.A7 (D-), J1.B7 (D-), U3.13 (USB_D-)
- new net IO20: J1.A6 (D+), J1.B6 (D+), U3.14 (USB_D+)
- new net IO6: R12.2, U3.6 (IO6)
- new net Q4: Q3.1 (G), Q4.3 (D), R14.1
- no-connect marks 24 -> 34
Other:
- note added: "Mounting Holes"
- note added: "USB Ports"
- note removed: "USB Power Only"
- moved on the sheet: C1, C3, C7, C8, J4, J5, R3, R4, R5, SW1, SW2, SW3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
