File: Hardware/PowerDistributionBoard.kicad_sch (KiCad schematic)
At the start: 62 parts, among them J1 USB_C_Programming_Port, J2 Main Input, J3 Main Output, J4 USB_A, J5 USB_C_Fast_Charging, J6 USB_C_Receptacle_PowerOnly_6P, Q1 2N7002(9V), Q2 2N7002(12V), Q3 AO3401A, Q4 2N7002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

Commit message: Uploading V1.0 Schematic pdf
Parts:
- removed H3: MountingHole, MountingHole:MountingHole_3.2mm_M3, symbol Mechanical:MountingHole
- removed J5: USB_C_Fast_Charging, Connector_USB:USB_C_Receptacle_HRO_TYPE-C-31-M-12, symbol Connector:USB_C_Receptacle_PowerOnly_6P
- removed R10, R11: R_Shunt, Resistor_SMD:R_2512_6332Metric_Pad1.40x3.35mm_HandSolder, symbol Device:R_Shunt
- removed SW3: SW_SPST, Button_Switch_THT:SW_Slide_SPDT_Straight_CK_OS102011MS2Q, symbol Switch:SW_SPST
- added J7: USB_C_Receptacle_USB2.0_16P, Connector_USB:USB_C_Receptacle_HRO_TYPE-C-31-M-12, symbol Connector:USB_C_Receptacle_USB2.0_16P
- added R10: Shunt_Main, Resistor_SMD:R_2512_6332Metric_Pad1.40x3.35mm_HandSolder, symbol Device:R
- added R11: Shunt_Vbus, Resistor_SMD:R_2512_6332Metric_Pad1.40x3.35mm_HandSolder, symbol Device:R
- added SW3: SW_SPDT, Button_Switch_THT:SW_Slide_SPDT_Straight_CK_OS102011MS2Q, symbol Switch:SW_SPDT
- SW1, SW2: footprint PDB-KiCad10:SW_PUSH_6x6mm_2Pin_P5.08mm -> 2_Pin_Button:SW_PUSH_6x6mm_2Pin_P5.08mm
Connections:
- net VBUS- is gone; now on net VBUS: U8.9 (Vin-)
- net VIN+ is gone; now on net +24V: U6.10 (Vin+), U6.8 (Vbus)
- net +24V: now also R10.1
- net GND: now also J7.A1 (GND), J7.A12 (GND), J7.B1 (GND), J7.B12 (GND), J7.SH (SHIELD)
- net VBUS: now also R11.2
- net VBUS+: now also C10.1, L2.2, R6.2, R11.1
- net VIN-: now also F1.2, R10.2
- net at C1.1, C3.1, F1.1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: now also SW3.2 (B)
- net at J3.1 (Pin_1), R17.1: now also SW3.1 (A)
- net at U4.1 (CC2), U4.14 (CC2): now also J7.B5 (CC2)
- net at U4.10 (CC1), U4.11 (CC1): now also J7.A5 (CC1)
- net at Q3.3 (D): now also J7.A4 (VBUS), J7.A9 (VBUS), J7.B4 (VBUS), J7.B9 (VBUS)
- no-connect marks 34 -> 41
Other:
- moved on the sheet: H4
